Commit message: add gripper control

File: project0/ros2-moveit2-arm-control/src/my_moveit_config/config/my_robot.ros2_control.xacro (robot description, xacro)
@@ -13,5 +13,4 @@
                   <param name="initial_value">${initial_positions['joint1']}</param>
                 </state_interface>
-                <state_interface name="velocity"/>
             </joint>
             <joint name="joint2">
@@ -20,5 +19,4 @@
                   <param name="initial_value">${initial_positions['joint2']}</param>
                 </state_interface>
-                <state_interface name="velocity"/>
             </joint>
             <joint name="joint3">
@@ -27,5 +25,4 @@
                   <param name="initial_value">${initial_positions['joint3']}</param>
                 </state_interface>
-                <state_interface name="velocity"/>
             </joint>
             <joint name="joint4">
@@ -34,5 +31,4 @@
                   <param name="initial_value">${initial_positions['joint4']}</param>
                 </state_interface>
-                <state_interface name="velocity"/>
             </joint>
             <joint name="joint5">
@@ -41,5 +37,4 @@
                   <param name="initial_value">${initial_positions['joint5']}</param>
                 </state_interface>
-                <state_interface name="velocity"/>
             </joint>
             <joint name="joint6">
@@ -48,5 +43,10 @@
                   <param name="initial_value">${initial_positions['joint6']}</param>
                 </state_interface>
-                <state_interface name="velocity"/>
+            </joint>
+            <joint name="gripper_left_finger_joint">
+                <command_interface name="position"/>
+                <state_interface name="position">
+                  <param name="initial_value">${initial_positions['gripper_left_finger_joint']}</param>
+                </state_interface>
             </joint>
         </ros2_control>
